File: RemoteLaunch_Controller/CameraTriggerRev 4_3 w Launch Controller 2023/CameraTriggerSensorNodeOnly.kicad_pcb (KiCad board)
At the start: 2 copper layers, 60 parts, among them IC1 3178, J1 Pwr switch, J10 SW, J11 pwr, J12 Screw_Terminal_01x02, J13 J13, J2 Camera 1 3.5mm, J3 Camera 2 3.5 mm, J4 Camera 1 Term, J5 Camera 2 Term, J6 qwiic, J7 In, J8 Out, J9 Misc, Q1 2n2222, Q2 MMBT3904, Q3 MMBT3904, Q4 2n2222, U1 AMS1117CD-5.0, U2 TLP291-4, U4 MCP23017T-E/SO, U5 ULN2803A

Commit message: Adding Rev4_3 rev
Parts:
- added H5: , MountingHole:MountingHole_3.7mm_Pad, F.Cu at (-94.0, 48.3)
- D1: value LED Trig -> D_1
- D6: value LED -> D_2
- J13: value J13 -> Screw_Terminal_01x02
- J9: value Misc -> Conn_01x09_Socket; footprint Connector_PinHeader_2.54mm:PinHeader_1x08_P2.54mm_Vertical -> Connector_PinHeader_2.54mm:PinHeader_1x09_P2.54mm_Vertical
- Q1, Q4: value 2n2222 -> 2SC1815; footprint Package_TO_SOT_THT:TO-18-3 -> Package_TO_SOT_SMD:SOT-23-3
- moved J9 6.37 mm to (-94.0, 40.6)
- moved Q4 3.75 mm to (-19.1, 84.8)
- moved TP1_GND1 2.86 mm to (-94.0, 12.7)
- moved Q1 2.35 mm to (-67.9, 86.9), turned to 90 degrees
Routing:
- net +3V3: track 175.6 -> 188.0 mm
- net Net-(Q4-B): track 3.75 -> 7.31 mm
- net Net-(J12-Pin_2): track 11.4 -> 15.0 mm
- net /Sheet621ECC97/MOSI: track 7.64 -> 9.70 mm
- net Net-(IC1-D0): track 7.64 -> 9.70 mm
- net /Sheet621ECC97/MISO: track 7.64 -> 9.70 mm
- net /Sheet621ECC97/A5: track 7.64 -> 9.70 mm
- net /Sheet621ECC97/A4: track 7.64 -> 9.70 mm
- net Net-(IC1-D1): track 7.64 -> 9.70 mm
- net /Sheet621ECC97/SCK: track 7.64 -> 9.66 mm
- net GND: track 58.3 -> 56.4 mm, vias 17 -> 20
- net Net-(Q1-B): track 5.16 -> 6.91 mm

Commit message: Fixing glitch in relay board;  Sending REv4_3 to fab
Changed lines of the file:
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@@
     (fp_line (start 1 0.6) (end 1 -0.6)
       (stroke (width 0.1) (type solid)) (layer "F.Fab"))
-    (pad "1" smd roundrect (at -1.025 0 180) (size 1.15 1.4) (layers "F.Cu" "F.Paste" "F.Mask") (roundrect_rratio 0.217391)
+    (pad "1" smd roundrect (at -1.025 0 180) (size 1.15 1.4) (layers "F.Cu" "F.Paste" "F.Mask") (roundrect_rratio 0.2173913043)
       (net 5 "Net-(D1-K)") (pinfunction "K") (pintype "passive"))
-    (pad "2" smd roundrect (at 1.025 0 180) (size 1.15 1.4) (layers "F.Cu" "F.Paste" "F.Mask") (roundrect_rratio 0.217391)
+    (pad "2" smd roundrect (at 1.025 0 180) (size 1.15 1.4) (layers "F.Cu" "F.Paste" "F.Mask") (roundrect_rratio 0.2173913043)
       (net 78 "D_1") (pinfunction "A") (pintype "passive"))
     (model "${KISYS3DMOD}/LED_SMD.3dshapes/LED_0805_2012Metric.wrl"
@@
     (fp_line (start 1 0.6) (end 1 -0.6)
       (stroke (width 0.1) (type solid)) (layer "F.Fab"))
-    (pad "1" smd roundrect (at -0.9625 0 180) (size 1.325 1.3) (layers "F.Cu" "F.Paste" "F.Mask") (roundrect_rratio 0.192308)
+    (pad "1" smd roundrect (at -0.9625 0 180) (size 1.325 1.3) (layers "F.Cu" "F.Paste" "F.Mask") (roundrect_rratio 0.1923076923)
       (net 10 "Net-(D4-K)") (pinfunction "K") (pintype "passive"))
-    (pad "2" smd roundrect (at 0.9625 0 180) (size 1.325 1.3) (layers "F.Cu" "F.Paste" "F.Mask") (roundrect_rratio 0.192308)
+    (pad "2" smd roundrect (at 0.9625 0 180) (size 1.325 1.3) (layers "F.Cu" "F.Paste" "F.Mask") (roundrect_rratio 0.1923076923)
       (net 7 "Shutter") (pinfunction "A") (pintype "passive"))
     (model "${KISYS3DMOD}/LED_SMD.3dshapes/LED_0805_2012Metric_Castellated.wrl"
@@
     (fp_line (start 1 0.6) (end 1 -0.6)
       (stroke (width 0.1) (type solid)) (layer "F.Fab"))
-    (pad "1" smd roundrect (at -1.025 0 180) (size 1.15 1.4) (layers "F.Cu" "F.Paste" "F.Mask") (roundrect_rratio 0.217391)
+    (pad "1" smd roundrect (at -1.025 0 180) (size 1.15 1.4) (layers "F.Cu" "F.Paste" "F.Mask") (roundrect_rratio 0.2173913043)
       (net 11 "Net-(D5-K)") (pinfunction "K") (pintype "passive"))
-    (pad "2" smd roundrect (at 1.025 0 180) (size 1.15 1.4) (layers "F.Cu" "F.Paste" "F.Mask") (roundrect_rratio 0.217391)
+    (pad "2" smd roundrect (at 1.025 0 180) (size 1.15 1.4) (layers "F.Cu" "F.Paste" "F.Mask") (roundrect_rratio 0.2173913043)
       (net 9 "Focus") (pinfunction "A") (pintype "passive"))
     (model "${KISYS3DMOD}/LED_SMD.3dshapes/LED_0805_2012Metric.wrl"
@@
     (fp_line (start 1 0.6) (end 1 -0.6)
       (stroke (width 0.1) (type solid)) (layer "F.Fab"))
-    (pad "1" smd roundrect (at -1.025 0 180) (size 1.15 1.4) (layers "F.Cu" "F.Paste" "F.Mask") (roundrect_rratio 0.217391)
+    (pad "1" smd roundrect (at -1.025 0 180) (size 1.15 1.4) (layers "F.Cu" "F.Paste" "F.Mask") (roundrect_rratio 0.2173913043)
       (net 23 "Net-(D6-K)") (pinfunction "K") (pintype "passive"))
-    (pad "2" smd roundrect (at 1.025 0 180) (size 1.15 1.4) (layers "F.Cu" "F.Paste" "F.Mask") (roundrect_rratio 0.217391)
+    (pad "2" smd roundrect (at 1.025 0 180) (size 1.15 1.4) (layers "F.Cu" "F.Paste" "F.Mask") (roundrect_rratio 0.2173913043)
       (net 79 "D_2") (pinfunction "A") (pintype "passive"))
     (model "${KISYS3DMOD}/LED_SMD.3dshapes/LED_0805_2012Metric.wrl"
@@
     (pad "4" smd roundrect (at 1.5 -2) (size 0.6 1.55) (layers "F.Cu" "F.Paste" "F.Mask") (roundrect_rratio 0.25)
       (net 27 "SCL_qwiic") (pinfunction "Pin_4") (pintype "passive"))
-    (pad "MP" smd roundrect (at -2.8 1.875) (size 1.2 1.8) (layers "F.Cu" "F.Paste" "F.Mask") (roundrect_rratio 0.208333))
-    (pad "MP" smd roundrect (at 2.8 1.875) (size 1.2 1.8) (layers "F.Cu" "F.Paste" "F.Mask") (roundrect_rratio 0.208333))
+    (pad "MP" smd roundrect (at -2.8 1.875) (size 1.2 1.8) (layers "F.Cu" "F.Paste" "F.Mask") (roundrect_rratio 0.2083333333))
+    (pad "MP" smd roundrect (at 2.8 1.875) (size 1.2 1.8) (layers "F.Cu" "F.Paste" "F.Mask") (roundrect_rratio 0.2083333333))
     (model "${KISYS3DMOD}/Connector_JST.3dshapes/JST_SH_SM04B-SRSS-TB_1x04-1MP_P1.00mm_Horizontal.wrl"
       (offset (xyz 0 0 0))
@@
     (fp_line (start 1 0.6) (end -1 0.6)
       (stroke (width 0.1) (type solid)) (layer "F.Fab"))
-    (pad "1" smd roundrect (at -1.025 0 90) (size 1.15 1.4) (layers "F.Cu" "F.Paste" "F.Mask") (roundrect_rratio 0.217391)
+    (pad "1" smd roundrect (at -1.025 0 90) (size 1.15 1.4) (layers "F.Cu" "F.Paste" "F.Mask") (roundrect_rratio 0.2173913043)
       (net 40 "Net-(J4-Pin_3)") (pintype "passive"))
-    (pad "2" smd roundrect (at 1.025 0 90) (size 1.15 1.4) (layers "F.Cu" "F.Paste" "F.Mask") (roundrect_rratio 0.217391)
+    (pad "2" smd roundrect (at 1.025 0 90) (size 1.15 1.4) (layers "F.Cu" "F.Paste" "F.Mask") (roundrect_rratio 0.2173913043)
       (net 48 "Net-(R9-Pad2)") (pintype "passive"))
     (model "${KISYS3DMOD}/Resistor_SMD.3dshapes/R_0805_2012Metric.wrl"
@@
     (fp_line (start 1 0.6) (end -1 0.6)
       (stroke (width 0.1) (type solid)) (layer "F.Fab"))
-    (pad "1" smd roundrect (at -1.025 0 90) (size 1.15 1.4) (layers "F.Cu" "F.Paste" "F.Mask") (roundrect_rratio 0.217391)
+    (pad "1" smd roundrect (at -1.025 0 90) (size 1.15 1.4) (layers "F.Cu" "F.Paste" "F.Mask") (roundrect_rratio 0.2173913043)
       (net 37 "Net-(J5-Pin_3)") (pintype "passive"))
-    (pad "2" smd roundrect (at 1.025 0 90) (size 1.15 1.4) (layers "F.Cu" "F.Paste" "F.Mask") (roundrect_rratio 0.217391)
+    (pad "2" smd roundrect (at 1.025 0 90) (size 1.15 1.4) (layers "F.Cu" "F.Paste" "F.Mask") (roundrect_rratio 0.2173913043)
       (net 49 "Net-(R10-Pad2)") (pintype "passive"))
     (model "${KISYS3DMOD}/Resistor_SMD.3dshapes/R_0805_2012Metric.wrl"
