File: RemoteLaunch_Controller/CameraTriggerRev 4_3 w Launch Controller 2023/Buzzer and Indicators.kicad_sch (KiCad schematic)
At the start: 9 parts, among them J12 Screw_Terminal_01x02, J13 Screw_Terminal_01x02, Q1 2n2222, Q4 2n2222

Commit message: Adding Rev4_3 rev
Parts:
- Q1: value 2n2222 -> 2SC1815; footprint Package_TO_SOT_THT:TO-18-3 -> Package_TO_SOT_SMD:SOT-23-3
- Q4: value 2n2222 -> 2SC1815; footprint Package_TO_SOT_THT:TO-18-3 -> Package_TO_SOT_SMD:SOT-23-3; LCSC (none) -> C181171
Changed lines of the file:
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@@
       (effects (font (size 1.27 1.27)) (justify left))
     )
-    (property "Value" "2n2222" (at 126.7714 105.283 0)
+    (property "Value" "2SC1815" (at 126.7714 105.283 0)
       (effects (font (size 1.27 1.27)) (justify left))
     )
-    (property "Footprint" "Package_TO_SOT_THT:TO-18-3" (at 127 106.045 0)
+    (property "Footprint" "Package_TO_SOT_SMD:SOT-23-3" (at 127 106.045 0)
       (effects (font (size 1.27 1.27) italic) (justify left) hide)
     )
@@
       (effects (font (size 1.27 1.27)) (justify left))
     )
-    (property "Value" "2n2222" (at 102.6414 170.053 0)
+    (property "Value" "2SC1815" (at 102.6414 170.053 0)
       (effects (font (size 1.27 1.27)) (justify left))
     )
-    (property "Footprint" "Package_TO_SOT_THT:TO-18-3" (at 102.87 170.815 0)
+    (property "Footprint" "Package_TO_SOT_SMD:SOT-23-3" (at 102.87 170.815 0)
       (effects (font (size 1.27 1.27) italic) (justify left) hide)
     )
@@
       (effects (font (size 1.27 1.27)) (justify left) hide)
     )
-    (property "LCSC" "" (at 97.79 168.91 0)
+    (property "LCSC" " C181171 " (at 97.79 168.91 0)
       (effects (font (size 1.27 1.27)) hide)
     )

Commit message: Working on adding polling / heartbeat;  Seem to have broken launch
Parts:
- Q1, Q4: footprint Package_TO_SOT_SMD:SOT-23-3 -> Package_TO_SOT_SMD:SOT-23
