File: RemoteLaunch_Controller/CameraTriggerRev 4_2 w Launch Controller 2023/CameraTriggerSensorNodeOnly.kicad_pcb (KiCad board)
At the start: 2 copper layers, 60 parts, among them IC1 3178, J1 Pwr switch, J10 SW, J11 pwr, J12 Screw_Terminal_01x02, J13 Screw_Terminal_01x02, J2 Camera 1 3.5mm, J3 Camera 2 3.5 mm, J4 Camera 1 Term, J5 Camera 2 Term, J6 qwiic, J7 In, J8 Out, J9 Misc, Q1 2SC1815, Q2 MMBT3904, Q3 MMBT3904, Q4 2SC1815, U1 AMS1117CD-5.0, U2 TLP291-4, U4 MCP23017T-E/SO, U5 ULN2803A

Commit message: Update to Kicad 7
Signed-off-by: Curtis Heisey <curtis.heisey@verizon.net>
Connections:
- net /Sheet621ECC97/~RST renamed /Sheet621ECC97/~{RST}
Other:
- net class Default removed
